File: System80RamEx.kicad_sch (KiCad schematic)
At the start: 23 parts, among them J1 Conn_01x08_Pin, J2 Conn_01x08_Pin, J3 Conn_01x08_Pin, J4 Conn_01x08_Pin, J5 Conn_01x08_Pin, J6 Conn_01x08_Pin, J7 Conn_01x08_Pin, J8 Conn_01x08_Pin, U1 KM62256CLP, U2 74LS04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

Commit message: Add files via upload
Cleaned up schematic
Connections:
- net D5 is gone; now on net D4: EC1.11 (Pin_11), Z3.15 (I2b), Z3.16 (O1a)
- net D6 is gone; now on net D4: EC1.18 (Pin_18), Z3.13 (I1b), Z3.14 (O2a)
- net D7 is gone; now on net D4: EC1.17 (Pin_17), Z3.11 (I0b), Z3.12 (O3a)
- net ~{DBIE} is gone; now on net D4: U6.8, Z2.1 (OEa), Z3.1 (OEa)
- net ~{DBOE} is gone; now on net D4: U5.8, Z2.19 (OEb), Z3.19 (OEb)
- net D4: now also U1.16 (Q4), U1.17 (Q5), U1.18 (Q6), U1.19 (Q7), Z3.2 (I0a), Z3.3 (O3b), Z3.4 (I1a), Z3.5 (O2b), Z3.6 (I2a), Z3.7 (O1b), Z3.8 (I3a), Z3.9 (O0b)
Other:
- moved on the sheet: EC1, J1, J2, J3, J4, J5, J6, J7, J8, RN1, RN2, RN3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
